Commit message: update moveit curi model

File: ros_assets/urdf/curi/urdf/curi.urdf (robot description, URDF)
Before this commit: robot curi, 42 links, 41 joints
Links:
- removed link world
Joints:
- removed joint reference

File: ros_assets/urdf/franka_description/robots/franka_panda.urdf (robot description, URDF)
Before this commit: robot panda, 11 links, 10 joints
Links:
- link panda_hand: geometry collision mesh filename=package://curi_goes_hands_on/ros_assets/urdf/franka_descrip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; visual mesh filename=package://curi_goes_hands_on/ros_assets/urdf/franka_descrip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
- link panda_leftfinger: geometry collision mesh filename=package://curi_goes_hands_on/ros_assets/urdf/franka_descrip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; visual mesh filename=package://curi_goes_hands_on/ros_assets/urdf/franka_descrip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
- link panda_link0: geometry collision mesh filename=package://curi_goes_hands_on/ros_assets/urdf/franka_descrip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; visual mesh filename=package://curi_goes_hands_on/ros_assets/urdf/franka_descrip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
- link panda_link1: geometry collision mesh filename=package://curi_goes_hands_on/ros_assets/urdf/franka_descrip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; visual mesh filename=package://curi_goes_hands_on/ros_assets/urdf/franka_descrip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
- link panda_link2: geometry collision mesh filename=package://curi_goes_hands_on/ros_assets/urdf/franka_descrip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; visual mesh filename=package://curi_goes_hands_on/ros_assets/urdf/franka_descrip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
- link panda_link3: geometry collision mesh filename=package://curi_goes_hands_on/ros_assets/urdf/franka_descrip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; visual mesh filename=package://curi_goes_hands_on/ros_assets/urdf/franka_descrip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
- link panda_link4: geometry collision mesh filename=package://curi_goes_hands_on/ros_assets/urdf/franka_descrip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; visual mesh filename=package://curi_goes_hands_on/ros_assets/urdf/franka_descrip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
- link panda_link5: geometry collision mesh filename=package://curi_goes_hands_on/ros_assets/urdf/franka_descrip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; visual mesh filename=package://curi_goes_hands_on/ros_assets/urdf/franka_descrip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
- link panda_link6: geometry collision mesh filename=package://curi_goes_hands_on/ros_assets/urdf/franka_descrip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; visual mesh filename=package://curi_goes_hands_on/ros_assets/urdf/franka_descrip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
- link panda_link7: geometry collision mesh filename=package://curi_goes_hands_on/ros_assets/urdf/franka_descrip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; visual mesh filename=package://curi_goes_hands_on/ros_assets/urdf/franka_descrip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
- link panda_rightfinger: geometry collision mesh filename=package://curi_goes_hands_on/ros_assets/urdf/franka_descrip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; visual mesh filename=package://curi_goes_hands_on/ros_assets/urdf/franka_descrip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
